File: meson.kicad_pcb (KiCad board)
At the start: 2 copper layers, 134.6 x 78.7 mm, 58 parts, among them K1 KEYSW, K10 KEYSW, K11 KEYSW, K12 KEYSW, K13 KEYSW, K14 KEYSW, K15 KEYSW, K16 KEYSW, K17 KEYSW, K18 KEYSW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

Commit message: tidy up and bom
Routing:
- net /col3: track 130.1 -> 128.5 mm
- net /row1: track 204.4 -> 203.8 mm
