File: PCB/meson.sch (KiCad schematic (older format))
At the start: 58 parts, among them K1 KEYSW, K10 KEYSW, K11 KEYSW, K12 KEYSW, K13 KEYSW, K14 KEYSW, K15 KEYSW, K16 KEYSW, K17 KEYSW, K18 KEYSW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

Commit message: "M3 mounting holes for pcb mounting+fixing big mistakes"
Parts:
- removed H1, H2: MountingHole, symbol Mechanical:MountingHole
Other:
- moved on the sheet: R1, R2, R3, RGB1, SW1, SW2, TRRS1, TRRS2, U1

Commit message: moving towards production
Parts:
- K1, K10, K11, K12, K13, K14, K15, K16, K17, K18, K19, K2, K20, K21, K22, K23, K3, K4, K5, K6, K7, K8, K9, Kb22: symbol keyboard_parts:KEYSW -> meson-rescue:KEYSW-keyboard_parts
Connections:
- net row0: now also U1.19 (F5); no longer U1.17 (F7)
- net row2: now also U1.16 (B1); no longer U1.18 (F6)
- net row3: now also U1.17 (F7); no longer U1.19 (F5)
Changed lines of the file:
@@
 SDA
 $Comp
-L keyboard_parts:KEYSW K1
+L meson-rescue:KEYSW-keyboard_parts K1
 U 1 1 5CA6F213
 P 4700 4200
@@
 $EndComp
 $Comp
-L keyboard_parts:KEYSW K2
+L meson-rescue:KEYSW-keyboard_parts K2
 U 1 1 5CA7405E
 P 5500 4200
@@
 $EndComp
 $Comp
-L keyboard_parts:KEYSW K3
+L meson-rescue:KEYSW-keyboard_parts K3
 U 1 1 5CA77280
 P 6300 4200
@@
 $EndComp
 $Comp
-L keyboard_parts:KEYSW K4
+L meson-rescue:KEYSW-keyboard_parts K4
 U 1 1 5CA77294
 P 7100 4200
@@
 $EndComp
 $Comp
-L keyboard_parts:KEYSW K5
+L meson-rescue:KEYSW-keyboard_parts K5
 U 1 1 5CA8AE62
 P 7900 4200
@@
 $EndComp
 $Comp
-L keyboard_parts:KEYSW K6
+L meson-rescue:KEYSW-keyboard_parts K6
 U 1 1 5CA8AE76
 P 8700 4200
@@
 $EndComp
 $Comp
-L keyboard_parts:KEYSW K23
+L meson-rescue:KEYSW-keyboard_parts K23
 U 1 1 5CA8AE9E
 P 8700 5650
@@
 $EndComp
 $Comp
-L keyboard_parts:KEYSW K8
+L meson-rescue:KEYSW-keyboard_parts K8
 U 1 1 5CAA2886
 P 4700 4700
@@
 $EndComp
 $Comp
-L keyboard_parts:KEYSW K9
+L meson-rescue:KEYSW-keyboard_parts K9
 U 1 1 5CAA289A
 P 5500 4700
@@
 $EndComp
 $Comp
-L keyboard_parts:KEYSW K10
-U 1 1 5CAA28AE
-P 6300 4700
-F 0 "K10" H 6300 4933 60  0000 C CNN
-F 1 "KEYSW" H 6300 4600 60  0001 C CNN
-F 2 "Keebio-Parts:MX-Alps-Choc-1U-NoLED-Reversible" H 6300 4700 60  0001 C CNN
-F 3 "" H 6300 4700 60  0000 C CNN
-	1    6300 4700
-	1    0    0    -1
-$EndComp
-$Comp
-L Diode:1N4148 D10
-U 1 1 5CAA28B8
-P 6000 4850
-F 0 "D10" V 6046 4771 50  0000 R CNN
-F 1 "1N4148" V 5955 4771 50  0000 R CNN
-F 2 "Diode_THT:D_DO-35_SOD27_P7.62mm_Horizontal" H 6000 4675 50  0001 C CNN
-F 3 "https://assets.nexperia.com/documents/data-sheet/1N4148_1N4448.pdf" H 6000 4850 50  0001 C CNN
-	1    6000 4850
-	0    -1   -1   0
-$EndComp
-$Comp
-L keyboard_parts:KEYSW K11
+L meson-rescue:KEYSW-keyboard_parts K11
 U 1 1 5CAA28C2
 P 7100 4700
@@
 $EndComp
 $Comp
-L keyboard_parts:KEYSW K12
+L meson-rescue:KEYSW-keyboard_parts K12
 U 1 1 5CAA28D6
 P 7900 4700
@@
 $EndComp
 $Comp
-L keyboard_parts:KEYSW K13
+L meson-rescue:KEYSW-keyboard_parts K13
 U 1 1 5CAA28EA
 P 8700 4700
@@
 $EndComp
 $Comp
-L keyboard_parts:KEYSW K14
+L meson-rescue:KEYSW-keyboard_parts K14
 U 1 1 5CAA28FE
 P 9500 4700
@@
 $EndComp
 $Comp
-L keyboard_parts:KEYSW K15
+L meson-rescue:KEYSW-keyboard_parts K15
 U 1 1 5CAAE14C
 P 4700 5200
@@
 $EndComp
 $Comp
-L keyboard_parts:KEYSW K16
+L meson-rescue:KEYSW-keyboard_parts K16
 U 1 1 5CAAE160
 P 5500 5200
@@
 $EndComp
 $Comp
-L keyboard_parts:KEYSW K17
-U 1 1 5CAAE174
-P 6300 5200
-F 0 "K17" H 6300 5433 60  0000 C CNN
-F 1 "KEYSW" H 6300 5100 60  0001 C CNN
-F 2 "Keebio-Parts:MX-Alps-Choc-1U-NoLED-Reversible" H 6300 5200 60  0001 C CNN
-F 3 "" H 6300 5200 60  0000 C CNN
-	1    6300 5200
-	1    0    0    -1
-$EndComp
-$Comp
 L Diode:1N4148 D17
 U 1 1 5CAAE17E
@@
 $EndComp
 $Comp
-L keyboard_parts:KEYSW K18
+L meson-rescue:KEYSW-keyboard_parts K18
 U 1 1 5CAAE188
 P 7100 5200
@@
 $EndComp
 $Comp
-L keyboard_parts:KEYSW K19
+L meson-rescue:KEYSW-keyboard_parts K19
 U 1 1 5CAAE19C
 P 7900 5200
@@
 $EndComp
 $Comp
-L keyboard_parts:KEYSW K20
+L meson-rescue:KEYSW-keyboard_parts K20
 U 1 1 5CAAE1B0
 P 8700 5200
@@
 $EndComp
 $Comp
-L keyboard_parts:KEYSW K21
+L meson-rescue:KEYSW-keyboard_parts K21
 U 1 1 5CAAE1C4
 P 9500 5200
@@
 $EndComp
 $Comp
-L keyboard_parts:KEYSW K22
+L meson-rescue:KEYSW-keyboard_parts K22
 U 1 1 5CABC8F4
 P 7900 5650
@@
 Wire Wire Line
 	4400 5000 5200 5000
-Connection ~ 5200 5000
-Wire Wire Line
-	5200 5000 6000 5000
-Connection ~ 6000 5000
-Wire Wire Line
-	6000 5000 6800 5000
-Connection ~ 6800 5000
 Wire Wire Line
 	6800 5000 7600 5000
@@
 	8400 5500 9200 5500
 $Comp
-L keyboard_parts:KEYSW Kb22
+L meson-rescue:KEYSW-keyboard_parts Kb22
 U 1 1 5CB2CEC6
 P 7900 5750
@@
 Wire Wire Line
 	7400 4700 7400 5200
-Wire Wire Line
-	6600 4200 6600 4700
-Connection ~ 6600 4700
-Wire Wire Line
-	6600 4700 6600 5200
 Wire Wire Line
 	5800 4200 5800 4700
@@
 	8400 6150 8400 5950
 $Comp
-L keyboard_parts:KEYSW K7
+L meson-rescue:KEYSW-keyboard_parts K7
 U 1 1 5CA8AE8A
 P 9500 4200
@@
 	8200 5650 8200 5750
 Connection ~ 8200 5650
-Text Label 7700 2550 0    50   ~ 0
+Text Label 7700 2750 0    50   ~ 0
 row2
-Text Label 7700 2450 0    50   ~ 0
+Text Label 7700 2650 0    50   ~ 0
 row3
 Text Label 7700 3050 0    50   ~ 0
@@
 Text Label 6300 2750 2    50   ~ 0
 col1
-Text Label 7700 2650 0    50   ~ 0
+Text Label 7700 2450 0    50   ~ 0
 row0
 Text Label 6300 2650 2    50   ~ 0
@@
 	4900 3350 5250 3350
 Connection ~ 4900 3350
+$Comp
+L Diode:1N4148 D10
+U 1 1 5CAA28B8
+P 6000 4850
+F 0 "D10" V 6046 4771 50  0000 R CNN
+F 1 "1N4148" V 5955 4771 50  0000 R CNN
+F 2 "Diode_THT:D_DO-35_SOD27_P7.62mm_Horizontal" H 6000 4675 50  0001 C CNN
+F 3 "https://assets.nexperia.com/documents/data-sheet/1N4148_1N4448.pdf" H 6000 4850 50  0001 C CNN
+	1    6000 4850
+	0    -1   -1   0
+$EndComp
+Connection ~ 5200 5000
+Connection ~ 6800 5000
+$Comp
+L meson-rescue:KEYSW-keyboard_parts K17
+U 1 1 5CAAE174
+P 6300 5200
+F 0 "K17" H 6300 5433 60  0000 C CNN
+F 1 "KEYSW" H 6300 5100 60  0001 C CNN
+F 2 "Keebio-Parts:MX-Alps-Choc-1U-NoLED-Reversible" H 6300 5200 60  0001 C CNN
+F 3 "" H 6300 5200 60  0000 C CNN
+	1    6300 5200
+	1    0    0    -1
+$EndComp
+Wire Wire Line
+	6600 4700 6600 5200
+Wire Wire Line
+	6600 4200 6600 4700
+Connection ~ 6600 4700
+$Comp
+L meson-rescue:KEYSW-keyboard_parts K10
+U 1 1 5CAA28AE
+P 6300 4700
+F 0 "K10" H 6300 4933 60  0000 C CNN
+F 1 "KEYSW" H 6300 4600 60  0001 C CNN
+F 2 "Keebio-Parts:MX-Alps-Choc-1U-NoLED-Reversible" H 6300 4700 60  0001 C CNN
+F 3 "" H 6300 4700 60  0000 C CNN
+	1    6300 4700
+	1    0    0    -1
+$EndComp
+Wire Wire Line
+	5200 5000 6000 5000
+Connection ~ 6000 5000
+Wire Wire Line
+	6000 5000 6800 5000
 $EndSCHEMATC
